File: splash_single_pcb_v1.kicad_sch (KiCad schematic)
At the start: 0 parts

Commit message: found stepper motor driver breakout from adafruit
Parts:
- added B1, B2, B3: (no value), splash_custom_footprints:A4988_breakout, symbol splash_symbols:A4988_borg
- added J1: Barrel_Jack, symbol Connector:Barrel_Jack
Other:
- note added: "Stepper Drivers"
